File: pcengine-rgb-addon.kicad_pcb (KiCad board)
At the start: 2 copper layers, 61.5 x 23.8 mm, 30 parts, among them J1 Conn_01x02_Male, U1 PCEngineExpansion, U2 THS7374, U3 Mini-DIN-9-Pin, U4 TS922A

Commit message: Initial Rev. C
Parts:
- removed J1: Conn_01x02_Male, Pin_Headers:Pin_Header_Straight_1x02_Pitch2.54mm
- removed R1: 10K, Resistors_SMD:R_0805_HandSoldering
- added C401: 10uF/Poly, Capacitor_SMD:CP_Elec_4x5.3, F.Cu at (133.9, 95.1)
- added C402: 10uF/Poly, Capacitor_SMD:CP_Elec_4x5.3, F.Cu at (128.9, 95.1)
- added C501: 220uF, Capacitor_Tantalum_SMD:CP_EIA-3528-12_Kemet-T_Pad1.50x2.35mm_HandSolder, F.Cu at (160.8, 93.2)
- added C601: 0.1uF, Capacitor_SMD:C_0603_1608Metric_Pad1.08x0.95mm_HandSolder, F.Cu at (120.5, 105.1)
- added C602: 0.1uF, Capacitor_SMD:C_0603_1608Metric_Pad1.08x0.95mm_HandSolder, F.Cu at (165.2, 99.2)
- added Q101: MMBT3906, Package_TO_SOT_SMD:SOT-23, F.Cu at (166.7, 94.1)
- added Q102: MMBT3904, Package_TO_SOT_SMD:SOT-23, F.Cu at (152.1, 92.8)
- added R101: 1K, Resistor_SMD:R_0603_1608Metric_Pad0.98x0.95mm_HandSolder, F.Cu at (156.6, 92.8)
- added R102: 1K, Resistor_SMD:R_0603_1608Metric_Pad0.98x0.95mm_HandSolder, F.Cu at (154.9, 92.8)
- added R103: 510R, Resistor_SMD:R_0603_1608Metric_Pad0.98x0.95mm_HandSolder, F.Cu at (149.2, 92.8)
- added R201: 2.2K, Resistor_SMD:R_0603_1608Metric_Pad0.98x0.95mm_HandSolder, F.Cu at (176.2, 92.1)
- added R202: 2.2K, Resistor_SMD:R_0603_1608Metric_Pad0.98x0.95mm_HandSolder, F.Cu at (174.3, 92.1)
- added R203: 2.2K, Resistor_SMD:R_0603_1608Metric_Pad0.98x0.95mm_HandSolder, F.Cu at (171.9, 92.1)
- added R204: 2.2K, Resistor_SMD:R_0603_1608Metric_Pad0.98x0.95mm_HandSolder, F.Cu at (170.1, 92.1)
- added R211: 2.2K, Resistor_SMD:R_0603_1608Metric_Pad0.98x0.95mm_HandSolder, F.Cu at (176.2, 95.6)
- added R212: 2.2K, Resistor_SMD:R_0603_1608Metric_Pad0.98x0.95mm_HandSolder, F.Cu at (174.3, 95.6)
- added R213: 2.2K, Resistor_SMD:R_0603_1608Metric_Pad0.98x0.95mm_HandSolder, F.Cu at (171.9, 95.6)
- added R214: 2.2K, Resistor_SMD:R_0603_1608Metric_Pad0.98x0.95mm_HandSolder, F.Cu at (170.1, 95.6)
- added R401: 1K, Resistor_SMD:R_0603_1608Metric_Pad0.98x0.95mm_HandSolder, F.Cu at (138.3, 98.8)
- added R402: 1K, Resistor_SMD:R_0603_1608Metric_Pad0.98x0.95mm_HandSolder, F.Cu at (124.6, 98.8)
- added R501: 75R, Resistor_SMD:R_0603_1608Metric_Pad0.98x0.95mm_HandSolder, F.Cu at (162.3, 97.2)
- C1, C10, C11, C2, C3, C4, C6, C7: footprint Capacitors_SMD:C_0805_HandSoldering -> Capacitor_SMD:C_0603_1608Metric_Pad1.08x0.95mm_HandSolder
- C12, C13: footprint Capacitors_SMD:CP_Elec_5x5.3 -> Capacitor_SMD:CP_Elec_4x5.3
- C5: footprint Capacitors_SMD:C_0805_HandSoldering -> Capacitor_SMD:C_0805_2012Metric_Pad1.18x1.45mm_HandSolder
- R10, R11, R12, R3, R4, R5, R6, R7, R8, R9: footprint Resistors_SMD:R_0805_HandSoldering -> Resistor_SMD:R_0603_1608Metric_Pad0.98x0.95mm_HandSolder
- R2: value 75R/Zero -> 1K; footprint Resistors_SMD:R_0805_HandSoldering -> Resistor_SMD:R_0603_1608Metric_Pad0.98x0.95mm_HandSolder
- U2: footprint Housings_SSOP:TSSOP-14_4.4x5mm_Pitch0.65mm -> Package_SO:TSSOP-14_4.4x5mm_P0.65mm
- moved U2 7.63 mm to (165.0, 103.0)
- moved C4 7.38 mm to (170.2, 99.8), turned to 90 degrees
- moved C2 6.68 mm to (171.4, 103.3)
- moved C1 6.31 mm to (171.4, 105.0)
- moved R3 5.84 mm to (137.3, 93.1)
- moved C6 5.51 mm to (139.2, 93.1)
- moved R7 5.36 mm to (138.3, 97.2), turned to 180 degrees
- moved C3 5.12 mm to (171.8, 99.8), turned to 90 degrees
- moved R6 4.26 mm to (124.6, 95.6), turned to 180 degrees
- moved R4 3.40 mm to (138.3, 95.6), turned to 0 degrees
- moved C12 2.23 mm to (144.1, 94.8), turned to 90 degrees
- moved R8 2.00 mm to (124.6, 97.2)
- moved C13 1.85 mm to (144.1, 102.5), turned to 90 degrees
- moved C5 1.82 mm to (165.3, 97.4)
- moved C11 1.27 mm to (118.2, 102.6)
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Connections:
- net Net-(C8-Pad1) renamed /CDA_L
- net Net-(C9-Pad1) renamed /CDA_R
- C1 pad 2: /Red_raw -> Net-(C1-Pad2)
- C2 pad 2: /Green_raw -> Net-(C2-Pad2)
- C3 pad 2: /Blue_raw -> Net-(C3-Pad2)
- C4 pad 2: /Video_raw -> Net-(C4-Pad2)
- R2 pad 1: /Sync -> Net-(Q101-Pad1)
- U1 pad A11: (no net) -> unconnected-(U1-PadA11)
- U1 pad A14: (no net) -> unconnected-(U1-PadA14)
- U1 pad B1: (no net) -> Net-(C402-Pad1)
- U1 pad B19: (no net) -> unconnected-(U1-PadB19)
- U1 pad B2: (no net) -> unconnected-(U1-PadB2)
- U1 pad B21: (no net) -> unconnected-(U1-PadB21)
- U1 pad B22: (no net) -> unconnected-(U1-PadB22)
- U1 pad B3: (no net) -> unconnected-(U1-PadB3)
- U1 pad B4: (no net) -> unconnected-(U1-PadB4)
- U1 pad B7: (no net) -> unconnected-(U1-PadB7)
- U1 pad C17: (no net) -> unconnected-(U1-PadC17)
- U1 pad C20: (no net) -> unconnected-(U1-PadC20)
- U1 pad C3: (no net) -> Net-(C401-Pad1)
- U1 pad C8: (no net) -> unconnected-(U1-PadC8)
- U2 pad 11: /Video -> Net-(R501-Pad2)
- U2 pad 12: /Blue -> /Red
- U2 pad 14: /Red -> /Blue
- U2 pad 7: (no net) -> unconnected-(U2-Pad7)
- U2 pad 8: (no net) -> unconnected-(U2-Pad8)
- U2 pad 9: Net-(J1-Pad2) -> +5V
- U3 pad 6: (no net) -> /Audio_Mono
Routing:
- net Net-(C402-Pad1): track 0.00 -> 15.1 mm
- net Net-(C1-Pad2): track 0.00 -> 14.2 mm
- net Net-(C401-Pad1): track 0.00 -> 13.2 mm
- net Net-(Q101-Pad2): track 0.00 -> 13.2 mm
- net Net-(C2-Pad2): track 0.00 -> 11.5 mm
- net Net-(J1-Pad2): track 10.1 -> 0.00 mm
- net /Sync: track 18.2 -> 8.25 mm
- net +5V: track 106.4 -> 113.5 mm
- net Net-(C4-Pad2): track 0.00 -> 6.89 mm
- net /Red_raw: track 17.6 -> 10.9 mm, vias 0 -> 1
- net /Green_raw: track 12.3 -> 5.59 mm
- net Net-(R501-Pad2): track 0.00 -> 6.73 mm
- net Net-(C3-Pad2): track 0.00 -> 6.62 mm
- net GNDA: track 26.1 -> 20.8 mm, vias 8 -> 15
- net /CDA_L: track 19.8 -> 24.8 mm, vias 0 -> 1
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Other:
- net class Default removed
- rule pad_to_mask_clearance: 0.2 -> 0
- board text added: "2023, Martin Hejnfelt (martin@hejnfelt.com)"
- board text added: "Attention! SCART Cable should contain 75 Ohm and 220uF capacitors on RGB lines!"
- board text added: "PCEngine RGB Add-on Rev. C"
- board text removed: "2018, Martin Hejnfelt (martin@hejnfelt.com)"
- board text removed: "Attention! SCART Cable should contain 75 Ohm and 220uF capacitors on video lines!"
- board text removed: "JP OFF=BYPASS JP ON=FILTER"
- board text removed: "PCEngine RGB Add-on"
